Commit message: Improve RViz fake robot feedback

File: ros/geekseek_fake_robot/urdf/geekseek_fake_robot.urdf.xacro (robot description, xacro)
@@ -4,4 +4,5 @@
   <material name="arm"><color rgba="0.18 0.55 0.88 1"/></material>
   <material name="accent"><color rgba="0.95 0.42 0.12 1"/></material>
+  <link name="world"/>
   <xacro:macro name="link_box" params="name size xyz material">
     <link name="${name}">
@@ -16,4 +17,7 @@
     <inertial><origin xyz="0 0 0.025"/><mass value="1"/><inertia ixx="0.003" ixy="0" ixz="0" iyy="0.003" iyz="0" izz="0.003"/></inertial>
   </link>
+  <joint name="world_to_base" type="fixed">
+    <parent link="world"/><child link="base_link"/>
+  </joint>
   <xacro:link_box name="shoulder_link" size="0.06 0.06 0.10" xyz="0 0 0.05" material="arm"/>
   <joint name="base_yaw_joint" type="revolute">

Commit message: Render STEP-based articulated robot in RViz

File: ros/geekseek_fake_robot/urdf/geekseek_fake_robot.urdf.xacro (robot description, xacro)
@@ -1,50 +1,77 @@
 <?xml version="1.0"?>
 <robot xmlns:xacro="http://www.ros.org/wiki/xacro" name="geekseek_fake_robot">
-  <material name="dark"><color rgba="0.10 0.12 0.15 1"/></material>
-  <material name="arm"><color rgba="0.18 0.55 0.88 1"/></material>
-  <material name="accent"><color rgba="0.95 0.42 0.12 1"/></material>
-  <link name="world"/>
-  <xacro:macro name="link_box" params="name size xyz material">
+  <material name="base"><color rgba="0.20 0.23 0.28 1"/></material>
+  <material name="link1"><color rgba="0.17 0.52 0.82 1"/></material>
+  <material name="link2"><color rgba="0.19 0.60 0.86 1"/></material>
+  <material name="link3"><color rgba="0.24 0.68 0.88 1"/></material>
+  <material name="link4"><color rgba="0.96 0.43 0.14 1"/></material>
+  <material name="tool"><color rgba="0.10 0.12 0.15 1"/></material>
+  <material name="kiosk"><color rgba="0.72 0.76 0.82 1"/></material>
+  <material name="screen"><color rgba="0.08 0.10 0.13 1"/></material>
+  <xacro:macro name="cad_link" params="name mesh material mass">
     <link name="${name}">
-      <visual><origin xyz="${xyz}"/><geometry><box size="${size}"/></geometry><material name="${material}"/></visual>
-      <collision><origin xyz="${xyz}"/><geometry><box size="${size}"/></geometry></collision>
-      <inertial><origin xyz="${xyz}"/><mass value="0.2"/><inertia ixx="0.001" ixy="0" ixz="0" iyy="0.001" iyz="0" izz="0.001"/></inertial>
+      <visual>
+        <geometry>
+          <mesh filename="package://geekseek_fake_robot/meshes/${mesh}" scale="0.001 0.001 0.001"/>
+        </geometry>
+        <material name="${material}"/>
+      </visual>
+      <inertial>
+        <mass value="${mass}"/>
+        <inertia ixx="0.01" ixy="0" ixz="0" iyy="0.01" iyz="0" izz="0.01"/>
+      </inertial>
     </link>
   </xacro:macro>
-  <link name="base_link">
-    <visual><origin xyz="0 0 0.025"/><geometry><cylinder radius="0.075" length="0.05"/></geometry><material name="dark"/></visual>
-    <collision><origin xyz="0 0 0.025"/><geometry><cylinder radius="0.075" length="0.05"/></geometry></collision>
-    <inertial><origin xyz="0 0 0.025"/><mass value="1"/><inertia ixx="0.003" ixy="0" ixz="0" iyy="0.003" iyz="0" izz="0.003"/></inertial>
+  <link name="world"/>
+  <link name="kiosk_link">
+    <visual>
+      <geometry><mesh filename="package://geekseek_fake_robot/meshes/kiosk_body.stl" scale="0.001 0.001 0.001"/></geometry>
+      <material name="kiosk"/>
+    </visual>
+    <visual>
+      <geometry><mesh filename="package://geekseek_fake_robot/meshes/ipad.stl" scale="0.001 0.001 0.001"/></geometry>
+      <material name="screen"/>
+    </visual>
+    <visual>
+      <geometry><mesh filename="package://geekseek_fake_robot/meshes/kiosk_camera.stl" scale="0.001 0.001 0.001"/></geometry>
+      <material name="tool"/>
+    </visual>
   </link>
+  <joint name="world_to_kiosk" type="fixed">
+    <parent link="world"/><child link="kiosk_link"/>
+  </joint>
+  <xacro:cad_link name="base_link" mesh="base_link.stl" material="base" mass="2.0"/>
   <joint name="world_to_base" type="fixed">
     <parent link="world"/><child link="base_link"/>
   </joint>
-  <xacro:link_box name="shoulder_link" size="0.06 0.06 0.10" xyz="0 0 0.05" material="arm"/>
+  <xacro:cad_link name="base_yaw_link" mesh="base_yaw_link.stl" material="link1" mass="1.5"/>
   <joint name="base_yaw_joint" type="revolute">
-    <parent link="base_link"/><child link="shoulder_link"/><origin xyz="0 0 0.05"/><axis xyz="0 0 1"/><limit lower="-2.8" upper="2.8" effort="10" velocity="1.5"/>
+    <parent link="base_link"/><child link="base_yaw_link"/>
+    <origin xyz="0 0 0.012"/><axis xyz="0 0 1"/>
+    <limit lower="-2.8" upper="2.8" effort="10" velocity="1.5"/>
   </joint>
-  <xacro:link_box name="upper_arm_link" size="0.045 0.045 0.16" xyz="0 0 0.08" material="arm"/>
+  <xacro:cad_link name="shoulder_link" mesh="shoulder_link.stl" material="link2" mass="1.5"/>
   <joint name="shoulder_pitch_joint" type="revolute">
-    <parent link="shoulder_link"/><child link="upper_arm_link"/><origin xyz="0 0 0.10"/><axis xyz="0 1 0"/><limit lower="-1.6" upper="1.6" effort="10" velocity="1.5"/>
+    <parent link="base_yaw_link"/><child link="shoulder_link"/>
+    <origin xyz="0 0 0.117"/><axis xyz="0 1 0"/>
+    <limit lower="-1.4" upper="1.4" effort="10" velocity="1.5"/>
   </joint>
-  <xacro:link_box name="forearm_link" size="0.04 0.04 0.14" xyz="0 0 0.07" material="arm"/>
+  <xacro:cad_link name="elbow_link" mesh="elbow_link.stl" material="link3" mass="1.5"/>
   <joint name="elbow_pitch_joint" type="revolute">
-    <parent link="upper_arm_link"/><child link="forearm_link"/><origin xyz="0 0 0.16"/><axis xyz="0 1 0"/><limit lower="-1.7" upper="1.7" effort="10" velocity="1.5"/>
+    <parent link="shoulder_link"/><child link="elbow_link"/>
+    <origin xyz="0 0 0.148"/><axis xyz="0 1 0"/>
+    <limit lower="-1.5" upper="1.5" effort="10" velocity="1.5"/>
   </joint>
-  <xacro:link_box name="wrist_yaw_link" size="0.05 0.05 0.05" xyz="0 0 0.025" material="accent"/>
-  <joint name="wrist_yaw_joint" type="revolute">
-    <parent link="forearm_link"/><child link="wrist_yaw_link"/><origin xyz="0 0 0.14"/><axis xyz="0 0 1"/><limit lower="-2.8" upper="2.8" effort="6" velocity="2"/>
+  <xacro:cad_link name="wrist_pitch_link" mesh="wrist_pitch_link.stl" material="link4" mass="1.2"/>
+  <joint name="wrist_pitch_joint" type="revolute">
+    <parent link="elbow_link"/><child link="wrist_pitch_link"/>
+    <origin xyz="0 0 0.108"/><axis xyz="0 1 0"/>
+    <limit lower="-1.5" upper="1.5" effort="8" velocity="1.8"/>
   </joint>
-  <xacro:link_box name="wrist_pitch_link" size="0.045 0.045 0.06" xyz="0 0 0.03" material="dark"/>
-  <joint name="wrist_pitch_joint" type="revolute">
-    <parent link="wrist_yaw_link"/><child link="wrist_pitch_link"/><origin xyz="0 0 0.05"/><axis xyz="0 1 0"/><limit lower="-1.5" upper="1.5" effort="6" velocity="2"/>
-  </joint>
-  <link name="camera_link">
-    <visual><origin xyz="0 0 0.025"/><geometry><box size="0.11 0.035 0.05"/></geometry><material name="dark"/></visual>
-    <collision><origin xyz="0 0 0.025"/><geometry><box size="0.11 0.035 0.05"/></geometry></collision>
-    <inertial><origin xyz="0 0 0.025"/><mass value="0.15"/><inertia ixx="0.001" ixy="0" ixz="0" iyy="0.001" iyz="0" izz="0.001"/></inertial>
-  </link>
-  <joint name="camera_roll_joint" type="revolute">
-    <parent link="wrist_pitch_link"/><child link="camera_link"/><origin xyz="0 0 0.06"/><axis xyz="1 0 0"/><limit lower="-1.57" upper="1.57" effort="4" velocity="2"/>
+  <xacro:cad_link name="end_effector_link" mesh="end_effector_link.stl" material="tool" mass="0.8"/>
+  <joint name="end_effector_yaw_joint" type="revolute">
+    <parent link="wrist_pitch_link"/><child link="end_effector_link"/>
+    <origin xyz="-0.108 0 -0.0205"/><axis xyz="0 0 1"/>
+    <limit lower="-2.8" upper="2.8" effort="6" velocity="2.0"/>
   </joint>
 </robot>
